File: dma-mapped-memory.kicad_sch (KiCad schematic)
At the start: 24 parts, among them U1 AS6C8008-55, U10 74LS157, U11 74LS157, U12 74LS157, U13 74LS157, U14 74LS157, U15 74LS04, U16 74LS373, U17 74LS373, U18 AS6C8008-55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

Commit message: add address registers
Other:
- added sheet Control Registers (registers.kicad_sch)
Changed lines of the file:
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@@
+    )
+  )
+  (sheet (at 339.09 19.05) (size 28.956 24.13) (fields_autoplaced)
+    (stroke (width 0.1524) (type solid))
+    (fill (color 0 0 0 0.0000))
+    (property "Sheetname" "Control Registers" (at 339.09 18.3384 0)
+      (effects (font (size 1.27 1.27)) (justify left bottom))
+    )
+    (property "Sheetfile" "registers.kicad_sch" (at 339.09 43.7646 0)
+      (effects (font (size 1.27 1.27)) (justify left top))
+    )
+    (instances
+      (project "dma-mapped-memory"
+        (path "/69886465-400e-42ab-8d15-9b306715bb96" (page "3"))
+      )
     )
   )

Commit message: simplify logic
Parts:
- removed unit 6 of U15
- removed unit 4 of U15
- removed unit 2 of U15
Connections:
- net AM10: now also U6.13 (CP), U6.6 (Q3)
- net ~{R}/W: now reaches U21.11 (LE)
- net ~{R}/W: now also U15.10, U17.1 (OE)
- net ~{DA20}: now reaches U19.6 (~{CE})
- net ~{DA20}: now also U15.2, U2.6 (~{CE})
- net ~{DA21}: now reaches U15.6, U2.40 (CE2)
- net ~{DA21}: now also U1.40 (CE2)
- net E: now reaches U2.41 (~{OE})
- net E: now also U1.41 (~{OE}), U18.41 (~{OE}), U19.41 (~{OE})
Other:
- moved on the sheet: U15C
