File: registers.kicad_sch (KiCad schematic)
At the start: 11 parts, among them U20 74HC08, U22 74HC21, U23 74HC02, U24 74HC21, U25 74HC04, U26 74HC375, U27 74HC375, U28 74HC375, U29 74HC375, U30 74HC21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

Commit message: simplify logic
Parts:
- removed U25, U31: 74HC04, Package_SO:SO-14_3.9x8.65mm_P1.27mm, symbol 74xx:74HC04
- added U15: 74LS04, Package_SO:SOIC-14_3.9x8.7mm_P1.27mm, symbol 74xx:74LS04
Connections:
- net D0: now also U28.7 (D1); no longer U28.1 (D0)
- net D1: now also U28.1 (D0); no longer U28.7 (D1)
- net D4: now also U29.7 (D1); no longer U29.1 (D0)
- net D5: now also U29.1 (D0); no longer U29.7 (D1)
- net PBA0: now also U28.5 (Q1); no longer U28.3 (Q0)
- net PBA1: now also U28.3 (Q0); no longer U28.5 (Q1)
- net PBA4: now also U29.5 (Q1); no longer U29.3 (Q0)
- net PBA5: now also U29.3 (Q0); no longer U29.5 (Q1)
- net ~{R}/W: now reaches U24.9
- net ~{R}/W: now also U30.9
- no-connect marks 29 -> 25
